File: ftdi.kicad_sch (KiCad schematic)
At the start: 43 parts

Commit message: Removed FTDI, added TPS65988 PD controller
Parts:
- removed C? (x14): C_100n_0402, antmicro-footprints:0402-cap, symbol antmicroCapacitors0402:C_100n_0402
- removed C? (x2): C_18p_0402, antmicro-footprints:0402-cap, symbol antmicroCapacitors0402:C_18p_0402
- removed C? (x2): C_10u_0603, antmicro-footprints:0603-cap, symbol antmicroCapacitors0603:C_10u_0603
- removed D? (x2): LG_L29K-G2J1-24-Z, antmicro-footprints:LED_0603, symbol antmicroLEDIndicationDiscrete:LG_L29K-G2J1-24-Z
- removed FB? (x3): BLM18PG330SH1D, antmicro-footprints:0603-res, symbol antmicroFerriteBeadsandChips:BLM18PG330SH1D
- removed R? (x5): R_0R_0402, antmicro-footprints:0402-res, symbol antmicroResistors0402:R_0R_0402
- removed R? (x2): R_1k_0402, antmicro-footprints:0402-res, symbol antmicroResistors0402:R_1k_0402
- removed R? (x2): R_100k_0402, antmicro-footprints:0402-res, symbol antmicroResistors0402:R_100k_0402
- removed R?: R_12k_0402, antmicro-footprints:0402-res, symbol antmicroResistors0402:R_12k_0402
- removed R? (x4): R_10k_0402, antmicro-footprints:0402-res, symbol antmicroResistors0402:R_10k_0402
- removed R? (x2): R_15k_0402, antmicro-footprints:0402-res, symbol antmicroResistors0402:R_15k_0402
- removed R?: R_2k_0402, antmicro-footprints:0402-res, symbol antmicroResistors0402:R_2k_0402
- removed U?: 93LC66BT-IMC, antmicro-footprints:DFN-8_2x3mm, symbol antmicroMemory:93LC66BT-IMC
- removed U?: FT4233HPQ, antmicro-footprints:QFN-76-1EP_9x9mm_P0.4mm_EP3.8x3.8mm, symbol antmicroInterfaceControllers:FT4233HPQ
- removed Y?: ABM8G-12.000MHZ-18-D2Y-T, antmicro-footprints:KX-7, symbol antmicroCrystals:ABM8G-12.000MHZ-18-D2Y-T
Connections:
- no-connect marks 33 -> 0
Other:
- note removed: "Config memory"
- note removed: "ORG: HIGH-x16 LOW-x8"
- note removed: "Orin Debug Interface"
- note removed: "PD1 Voltage sensing"
- note removed: "PD2 Voltage Sensing"
- note removed: "Power configuration for PD"
- note removed: "USB2 Orientation detection: high-CC1, low-CC2"
