File: peripherals.kicad_sch (KiCad schematic)
At the start: 69 parts, among them J1 ERF8-040-05.0-L-DV-K-TR, J801 TC2050-IDC-NL, J803 533980471, Q801 BSS138W-7-F, Q802 BSS138W-7-F, Q803 BSS138W-7-F, Q804 BSS138W-7-F, U803 PCAL6416AHF, U805 AP22615, U806 AP22615, U807 74LVC1T45GM

Commit message: Added 12V to the expansion connector, changed connector pinout
Parts:
- removed C808, C809: C_100n_0402, antmicro-footprints:0402-cap, symbol antmicroCapacitors0402:C_100n_0402
- removed C9, C?: C_1u_0402, antmicro-footprints:0402-cap, symbol antmicroCapacitors0402:C_1u_0402
- removed D803: LTST-C190GKT, antmicro-footprints:LED_0603, symbol antmicroLEDIndicationDiscrete:LTST-C190GKT
- removed Q804: BSS138W-7-F, antmicro-footprints:SOT-323, symbol antmicroTransistorsFETsMOSFETsSingle:BSS138W-7-F
- removed R817: R_0R_0402, antmicro-footprints:0402-res, symbol antmicroResistors0402:R_0R_0402
- removed R820: R_100k_0402, antmicro-footprints:0402-res, symbol antmicroResistors0402:R_100k_0402
- removed R821, R822: R_10k_0402, antmicro-footprints:0402-res, symbol antmicroResistors0402:R_10k_0402
- removed R824, R825: R_4k7_0402, antmicro-footprints:0402-res, symbol antmicroResistors0402:R_4k7_0402
- removed R829: R_200R_0603, antmicro-footprints:0603-res, symbol antmicroResistors0603:R_200R_0603
- removed TP801, TP802: TP_SMD_0_75MM, antmicro-footprints:Testpoint_smd_0_75mm, symbol antmicroTestPoints:TP_SMD_0_75MM
- removed U805, U806: AP22615, antmicro-footprints:TSOT23-6, symbol antmicroPMICPowerDistributionSwitchesLoadDrivers:AP22615
- added C? (x4): C_1u_0402, antmicro-footprints:0402-cap, symbol antmicroCapacitors0402:C_1u_0402
- added R? (x4): R_0R_0603, antmicro-footprints:0603-res, symbol antmicroResistors0603:R_0R_0603
Connections:
- net +3V3: now also R?.2
- net +5V: now also R?.1
- net 3V3_STDB: now also R?.2; no longer J1.76
- net CAN_RX: now also J1.68; no longer J1.65
- net CAN_TX: now also J1.70; no longer J1.67
- net EXT_GPIO0: no longer J1.31
- net EXT_GPIO1: no longer J1.33
- net EXT_GPIO2: no longer J1.35
- net EXT_GPIO3: no longer J1.36
- net EXT_GPIO4: no longer J1.40
- net GND: now also J1.71, J1.72, J1.76, C?.2, C?.2, C?.2, C?.2; no longer J1.74
- net GPIO01: now also J1.31; no longer J1.39
- net GPIO07: now also J1.33; no longer J1.41
- net GPIO09: now also J1.35; no longer J1.43
- net GPIO10: now also J1.39; no longer J1.45
- net GPIO11: now also J1.42; no longer J1.47
- net GPIO12: now also J1.40; no longer J1.42
- net GPIO13: now also J1.36; no longer J1.44
- net I2C2_SCL: now also J1.66; no longer J1.48
- net I2C2_SDA: now also J1.64; no longer J1.46
- net I2S0_LRCK: now also J1.47; no longer J1.72
- net I2S0_SCLK: now also J1.46; no longer J1.66
- net I2S0_SDIN: now also J1.45; no longer J1.70
- net I2S0_SDOUT: now also J1.48; no longer J1.68
- net SYS_SCL: now also J1.65; no longer J1.64
- net UART0_RXD: now also J1.43; no longer J1.71
- net UART0_TXD: now also J1.41; no longer J1.69
- net 1V8_CONN: now reaches J1.73, R?.1
- net 1V8_CONN: now also C?.1
- net CONN_3V3 renamed 12V_CONN
- net 12V_CONN: now also C?.1, R?.2
- net CONN_5V renamed 5V_CONN
- net 5V_CONN: now also R?.2
- net GPIOEX_P0_6: no longer names the net of U803.7 (P0_6)
- new net +12V: R?.1
- new net 3V3_CONN: C?.1, J1.67, J1.69, R?.1
- new net 3V3_STDB_CONN: C?.1, J1.74, R?.1
- new net GPIO00: J1.44
Other:
- note removed: "CONN_PWR"
- moved on the sheet: C1, C2, C3, C4, C5, C6, C7, C804, C810, C812, D801, D802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
