File: peripherals.kicad_sch (KiCad schematic)
At the start: 81 parts, among them J10 533980471, J11 ERF8-040-05.0-L-DV-K-TR, J9 TC2050-IDC-NL, Q10 NX138BKMYL, Q9 NX138BKMYL, U30 TPD4E05U06QDQARQ1, U33 NTS0102GT, U34 PCAL6408ABSHP

Commit message: Fix symbols after loclib
Connections:
- net CSIA_PEN: now also R25.1
- net CSIB_PEN: now also R25.2
- net DISABLE_POE_DCDC: now also R25.4
- net GPIOEX_P0_0: now also R25.8
- net GPIOEX_P0_1: now also R25.7
- net GPIOEX_P0_2: now also R25.6
- net GPIOEX_P0_3: now also R25.5
- net USBC1_PEN: now also R25.3
