File: jetson-orin-baseboard.kicad_pcb (KiCad board)
At the start: 8 copper layers, 110 x 55 mm, 646 parts, among them IC1 ACPL-217-500E, J1 2199230-6, J10 533980471, J11 ERF8-040-05.0-L-DV-K-TR, J12 1053131102, J13 46756-1001, J2 1-2199230-6, J3 USB4105-GF-A, J4 WE_632723300011_alt_symbol, J5 WE_632723300011_alt_symbol, J6 5-2337992-8, J7 WE_68715014522, J8 WE_68715014522, J9 TC2050-IDC-NL, M1 jetson-orin-nx/nano-module, M2 M2_4222, M3 M2_2280, Q1 BSS138W-7-F, Q10 BSS138W-7-F, Q11 BSS138W-7-F, Q12 BSS138W-7-F, Q13 BCM857BS-7-F, Q14 BCM857BS-7-F, Q15 SSM3J332R, Q16 SSM3J332R, Q17 BSS138W-7-F, Q18 BSS138W-7-F, Q19 BSS138W-7-F, Q2 BSS138W-7-F, Q20 BSS138W-7-F, Q21 BSS138APW, Q3 BSS138W-7-F, Q4 BSS138W-7-F, Q5 BSS138W-7-F, Q6 BSS138W-7-F, Q7 BSS138W-7-F, Q8 BSS138W-7-F, Q9 BSS138W-7-F, SW1 PCM12SMTR, U1 74LVC1T45GM, U10 TUSB1046-DCI, U11 TPD4E05U06QDQARQ1, U12 AP22615, U13 TPD4E05U06QDQARQ1, U14 TPD4E05U06QDQARQ1, U15 TPD4E05U06QDQARQ1, U16 TPD4E05U06QDQARQ1, U17 HD3SS3220, U18 AP22615, U19 TPD4E05U06QDQARQ1, U2 74LVC2G07GV, U20 TPD4E05U06QDQARQ1, U21 TPD4E05U06QDQARQ1, U22 TPS2372-3RGWR, U23 ULS-12/5-D48N-C, U24 AP22615, U25 AP22615, U26 PCA9547BS, U27 NX3DV642, U28 NX3DV642, U29 AP22615, U3 74LVC2G07GV, U30 AP22615, U31 NTS0102GT, U32 NTS0102GT, U33 74LVC1T45GM, U34 PCAL6408ABSHP, U37 74LVC2G14GV, U38 74LVC1G175GV, U39 MP2386GG-P, U40 MP2386GG-P, U41 TPS7B8133DRVR, U42 TPS7A0518PDBVT, U43 NTS0102GT, U44 TPD4E02B04DQA, U45 TPD4E02B04DQA, U46 TPD4E02B04DQA, U5 FT230XQ-R, U6 TPS65988, U7 W25Q80DVUXIE_TR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

Commit message: Prepare more advanced mockup setup
Parts:
- removed BAT1: MS621FE-FL11E, antmicro-footprints:MS621FE-FL11E
- removed C100, C101, C104, C108, C109, C110, C111, C112, C113, C118, C119, C124, C45, C7, C8, C87, C88, C89, C90, C91, C96, C97: C_100n_0402, antmicro-footprints:0402-cap
- removed C105, C106, C107, C114, C115, C142: C_1u_0402, antmicro-footprints:0402-cap
- removed C116, C117, C137, C34: C_10u_0402, antmicro-footprints:0402-cap
- removed C131: C_2u2_0402, antmicro-footprints:0402-cap
- removed C134, C32: C_10u_25V_0603, antmicro-footprints:0603-cap
- removed C79: C_22u_2220_100V, antmicro-footprints:2220-cap
- removed D26, D27, D8: LTST-C190GKT, antmicro-footprints:LED_0603
- removed D28: DF2S30FS, antmicro-footprints:SOD-923
- removed D30, D31: ESD9X5.0ST5G, antmicro-footprints:SOD-923
- removed D34, D36, D37: RB521S30T1G, antmicro-footprints:SOD-523
- removed J11: ERF8-040-05.0-L-DV-K-TR, antmicro-footprints:ERF8-040-XX.X-X-DV-XX
- removed J12: 1053131102, antmicro-footprints:1053131102
- removed Q1, Q10, Q11, Q12, Q17, Q18, Q19, Q2, Q20, Q9: BSS138W-7-F, antmicro-footprints:SOT-323
- removed Q13, Q14: BCM857BS-7-F, antmicro-footprints:SOT-363
- removed Q15, Q16: SSM3J332R, antmicro-footprints:SOT-23-3
- removed R105, R159, R180, R222, R230, R249, R262: R_100k_0402, antmicro-footprints:0402-res
- removed R106: R_200R_0603, antmicro-footprints:0603-res
- removed R13, R15, R16, R161, R162, R166, R167, R168, R17, R171, R174, R179, R18, R211, R212, R213, R214, R215, R216, R217, R218, R224, R225, R226, R227, R228, R229, R236, R237, R238, R239, R240, R241, R243, R244, R245, R246, R260, R268, R40, R60, R61, R76: R_0R_0402, antmicro-footprints:0402-res
- removed R158, R160, R169, R170, R172, R173, R177, R178, R294, R78: R_2k2_0402, antmicro-footprints:0402-res
- removed R163, R164, R165, R183, R184, R220, R250, R251, R254, R255, R259, R47, R49, R74, R77: R_10k_0402, antmicro-footprints:0402-res
- removed R175, R176, R185, R186: R_4k7_0402, antmicro-footprints:0402-res
- removed R219: R_10k2_0402, antmicro-footprints:0402-res
- removed R223, R231: R_200R_0402, antmicro-footprints:0402-res
- removed R233, R234, R235, R247, R248, R273, R276: R_0R_0603, antmicro-footprints:0603-res
- removed R252, R253: R_0R_1206, antmicro-footprints:1206-res
- removed R256: R_1k_0402, antmicro-footprints:0402-res
- removed R257, R258, R261: R_200k_0402, antmicro-footprints:0402-res
- removed R265: R_5R6_0402, antmicro-footprints:0402-res
- removed R37, R38: R_47k_0402, antmicro-footprints:0402-res
- removed S4, S5: B3U-3000PM, antmicro-footprints:B3U-3000P
- removed TP1, TP10, TP11, TP12, TP13, TP14, TP15, TP16, TP17, TP18, TP19, TP2, TP20, TP21, TP22, TP23, TP24, TP25, TP26, TP27, TP29, TP3, TP30, TP31, TP32, TP33, TP34, TP35, TP36, TP37, TP38, TP39, TP4, TP40, TP41, TP42, TP43, TP44, TP45, TP46, TP47, TP48, TP49, TP5, TP50, TP51, TP52, TP53, TP54, TP55, TP56, TP57, TP6, TP7, TP8, TP9: TP_SMD_0_75MM, antmicro-footprints:Testpoint_smd_0_75mm
- removed U2, U3: 74LVC2G07GV, antmicro-footprints:SC-74
- removed U24, U25, U29, U30, U9: AP22615, antmicro-footprints:TSOT23-6
- removed U26: PCA9547BS, antmicro-footprints:VQFN-24
- removed U31, U32: NTS0102GT, antmicro-footprints:PSON50P100X195X50-8N
- removed U34: PCAL6408ABSHP, antmicro-footprints:VQFN-16-1EP_3x3mm
- removed U37: 74LVC2G14GV, antmicro-footprints:SOT23-6L
- removed U38: 74LVC1G175GV, antmicro-footprints:SOT-23-6
- removed U41, U8: TPS7B8133DRVR, antmicro-footprints:WSON6_TI_2x2mm
- removed U42: TPS7A0518PDBVT, antmicro-footprints:SOT-23-5
- removed kibuzzard-633EE390: G***, kibuzzard-633EE390
- added REF**: SAMTEC_LSHM-140-01-L-DH-A-S-TR, antmicro-footprints:SAMTEC_LSHM-140-01-L-DH-A-S-TR, B.Cu at (139.4, 97.4)
- C102, C103, C145, C146, C147, C148, C149, C150, C151, C152, C153, C154, C155, C156, C157, C158, C159, C160, C161, C162, C26, C28, C30, C33, C35, C53, C58, C59, C92, C93, D1, D16, D17, D19, D21, D22, D23, D35, D4, D5, J9, Q5, Q6, Q7, Q8, R181, R182, R187, R188, R189, R190, R191, R192, R193, R195, R196, R198, R203, R204, R221, R277, R278, R39, R41, R42, R43, R44, R45, R48, R50, R51, R52, R53, R54, R55, R62, R63, R64, R65, R66, R67, R68, R69, R70, R71, SW1, U27, U28, U33, U6, U7: moved to B.Cu
- J7, S1, S2, S3: moved to F.Cu
- moved R14 293.1 mm to (125.8, 98.5), turned to 180 degrees
- moved R28 292.3 mm to (125.8, 97.5), turned to 180 degrees
- moved C10 291.0 mm to (125.8, 95.5), turned to 180 degrees
- moved C9 290.3 mm to (125.8, 94.5), turned to 180 degrees
- moved R26 283.9 mm to (126.2, 83.7), turned to 90 degrees
- moved R25 281.9 mm to (125.2, 83.7), turned to 90 degrees
- moved J1 275.7 mm to (118.2, 94.0), turned to -90 degrees
- moved C12 274.3 mm to (113.6, 102.8), turned to 180 degrees
- moved R31 272.3 mm to (113.7, 100.2), turned to 180 degrees
- moved R30 271.4 mm to (113.7, 99.2), turned to 180 degrees
- moved R27 269.8 mm to (113.5, 97.5), turned to 0 degrees
- moved R35 266.9 mm to (113.8, 93.3), turned to 180 degrees
- moved R36 266.2 mm to (113.8, 92.3), turned to 180 degrees
- moved R33 265.4 mm to (113.8, 91.3), turned to 180 degrees
- moved R34 264.7 mm to (113.8, 90.3), turned to 180 degrees
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
Commit message: Recover all components placement
Parts:
- removed REF**: SAMTEC_LSHM-140-01-L-DH-A-S-TR, antmicro-footprints:SAMTEC_LSHM-140-01-L-DH-A-S-TR
- added BAT1: MS621FE-FL11E, antmicro-footprints:MS621FE-FL11E, B.Cu at (60.9, 64.8)
- added C100: C_100n_0402, antmicro-footprints:0402-cap, F.Cu at (117.6, 142.8)
- added C101: C_100n_0402, antmicro-footprints:0402-cap, F.Cu at (111.6, 142.8)
- added C104: C_100n_0402, antmicro-footprints:0402-cap, F.Cu at (148.1, 169.7)
- added C105: C_1u_0402, antmicro-footprints:0402-cap, F.Cu at (151.4, 109.5)
- added C106: C_1u_0402, antmicro-footprints:0402-cap, F.Cu at (151.4, 111.5)
- added C107: C_1u_0402, antmicro-footprints:0402-cap, F.Cu at (151.4, 114.1)
- added C108: C_100n_0402, antmicro-footprints:0402-cap, F.Cu at (150.8, 85.5)
- added C109: C_100n_0402, antmicro-footprints:0402-cap, F.Cu at (159.2, 86.3)
- added C110: C_100n_0402, antmicro-footprints:0402-cap, F.Cu at (159.2, 87.3)
- added C111: C_100n_0402, antmicro-footprints:0402-cap, F.Cu at (159.2, 92.1)
- added C112: C_100n_0402, antmicro-footprints:0402-cap, F.Cu at (150.8, 86.5)
- added C113: C_100n_0402, antmicro-footprints:0402-cap, F.Cu at (159.2, 91.1)
- added C114: C_1u_0402, antmicro-footprints:0402-cap, F.Cu at (158.6, 111.5)
- added C115: C_1u_0402, antmicro-footprints:0402-cap, F.Cu at (158.6, 114.1)
- added C116: C_10u_0402, antmicro-footprints:0402-cap, F.Cu at (111.8, 171.3)
- added C117: C_10u_0402, antmicro-footprints:0402-cap, F.Cu at (111.2, 172.8)
- added C118: C_100n_0402, antmicro-footprints:0402-cap, F.Cu at (117.8, 171.7)
- added C119: C_100n_0402, antmicro-footprints:0402-cap, F.Cu at (119.2, 171.2)
- added C124: C_100n_0402, antmicro-footprints:0402-cap, F.Cu at (127.7, 171.7)
- added C131: C_2u2_0402, antmicro-footprints:0402-cap, F.Cu at (78.2, 161.5)
- added C134: C_10u_25V_0603, antmicro-footprints:0603-cap, F.Cu at (28.2, 159.7)
- added C137: C_10u_0402, antmicro-footprints:0402-cap, F.Cu at (32.0, 159.8)
- added C142: C_1u_0402, antmicro-footprints:0402-cap, F.Cu at (78.2, 159.5)
- added C32: C_10u_25V_0603, antmicro-footprints:0603-cap, F.Cu at (54.1, 147.1)
- added C34: C_10u_0402, antmicro-footprints:0402-cap, F.Cu at (58.9, 146.5)
- added C45: C_100n_0402, antmicro-footprints:0402-cap, F.Cu at (103.3, 196.9)
- added C7: C_100n_0402, antmicro-footprints:0402-cap, F.Cu at (56.6, 201.0)
- added C79: C_22u_2220_100V, antmicro-footprints:2220-cap, B.Cu at (41.2, 96.2)
- added C8: C_100n_0402, antmicro-footprints:0402-cap, F.Cu at (56.6, 205.0)
- added C87: C_100n_0402, antmicro-footprints:0402-cap, F.Cu at (90.2, 196.9)
- added C88: C_100n_0402, antmicro-footprints:0402-cap, F.Cu at (96.2, 196.9)
- added C89: C_100n_0402, antmicro-footprints:0402-cap, F.Cu at (131.8, 197.2)
- added C90: C_100n_0402, antmicro-footprints:0402-cap, F.Cu at (78.2, 196.8)
- added C91: C_100n_0402, antmicro-footprints:0402-cap, F.Cu at (84.2, 196.9)
- added C96: C_100n_0402, antmicro-footprints:0402-cap, F.Cu at (114.0, 142.8)
- added C97: C_100n_0402, antmicro-footprints:0402-cap, F.Cu at (108.0, 142.8)
- added D26: LTST-C190GKT, antmicro-footprints:LED_0603, F.Cu at (138.4, 212.7)
- added D27: LTST-C190GKT, antmicro-footprints:LED_0603, F.Cu at (146.4, 212.7)
- added D28: DF2S30FS, antmicro-footprints:SOD-923, F.Cu at (80.3, 178.1)
- added D30: ESD9X5.0ST5G, antmicro-footprints:SOD-923, F.Cu at (31.0, 157.8)
- added D31: ESD9X5.0ST5G, antmicro-footprints:SOD-923, F.Cu at (81.2, 157.7)
- added D34: RB521S30T1G, antmicro-footprints:SOD-523, B.Cu at (60.4, 61.6)
- added D36: RB521S30T1G, antmicro-footprints:SOD-523, F.Cu at (111.4, 167.0)
- added D37: RB521S30T1G, antmicro-footprints:SOD-523, F.Cu at (107.4, 172.4)
- added D8: LTST-C190GKT, antmicro-footprints:LED_0603, F.Cu at (123.9, 222.2)
- added J11: ERF8-040-05.0-L-DV-K-TR, antmicro-footprints:ERF8-040-XX.X-X-DV-XX, F.Cu at (155.0, 97.9)
- added J12: 1053131102, antmicro-footprints:1053131102, F.Cu at (-5.95, 112.7)
- added Q1: BSS138W-7-F, antmicro-footprints:SOT-323, F.Cu at (39.3, 189.8)
- added Q10: BSS138W-7-F, antmicro-footprints:SOT-323, F.Cu at (136.2, 212.5)
- added Q11: BSS138W-7-F, antmicro-footprints:SOT-323, F.Cu at (144.2, 212.5)
- added Q12: BSS138W-7-F, antmicro-footprints:SOT-323, F.Cu at (111.2, 169.3)
- added Q13: BCM857BS-7-F, antmicro-footprints:SOT-363, F.Cu at (79.5, 176.2)
- added Q14: BCM857BS-7-F, antmicro-footprints:SOT-363, F.Cu at (79.4, 169.2)
- added Q15: SSM3J332R, antmicro-footprints:SOT-23-3, F.Cu at (82.9, 176.2)
- added Q16: SSM3J332R, antmicro-footprints:SOT-23-3, F.Cu at (82.8, 169.2)
- added Q17: BSS138W-7-F, antmicro-footprints:SOT-323, F.Cu at (118.2, 173.7)
- added Q18: BSS138W-7-F, antmicro-footprints:SOT-323, F.Cu at (42.6, 165.0)
- added Q19: BSS138W-7-F, antmicro-footprints:SOT-323, F.Cu at (127.7, 173.8)
- added Q2: BSS138W-7-F, antmicro-footprints:SOT-323, F.Cu at (120.9, 222.2)
- added Q20: BSS138W-7-F, antmicro-footprints:SOT-323, F.Cu at (45.7, 165.0)
- added Q9: BSS138W-7-F, antmicro-footprints:SOT-323, F.Cu at (152.2, 191.6)
- added R105: R_100k_0402, antmicro-footprints:0402-res, F.Cu at (118.9, 222.1)
- added R106: R_200R_0603, antmicro-footprints:0603-res, F.Cu at (126.7, 222.2)
- added R13: R_0R_0402, antmicro-footprints:0402-res, F.Cu at (50.5, 204.5)
- added R15: R_0R_0402, antmicro-footprints:0402-res, F.Cu at (159.2, 95.1)
- added R158: R_2k2_0402, antmicro-footprints:0402-res, F.Cu at (130.6, 192.2)
- added R159: R_100k_0402, antmicro-footprints:0402-res, F.Cu at (96.1, 193.4)
- added R16: R_0R_0402, antmicro-footprints:0402-res, F.Cu at (51.0, 203.0)
- added R160: R_2k2_0402, antmicro-footprints:0402-res, F.Cu at (129.6, 192.2)
- added R161: R_0R_0402, antmicro-footprints:0402-res, F.Cu at (133.3, 198.8)
- added R162: R_0R_0402, antmicro-footprints:0402-res, F.Cu at (133.3, 199.8)
- added R163: R_10k_0402, antmicro-footprints:0402-res, F.Cu at (132.4, 195.6)
- added R164: R_10k_0402, antmicro-footprints:0402-res, F.Cu at (94.8, 198.9)
- added R165: R_10k_0402, antmicro-footprints:0402-res, F.Cu at (100.8, 198.9)
- added R166: R_0R_0402, antmicro-footprints:0402-res, F.Cu at (132.1, 191.7)
- added R167: R_0R_0402, antmicro-footprints:0402-res, F.Cu at (133.3, 197.8)
- added R168: R_0R_0402, antmicro-footprints:0402-res, F.Cu at (133.3, 196.7)
- added R169: R_2k2_0402, antmicro-footprints:0402-res, F.Cu at (128.6, 192.2)
- added R17: R_0R_0402, antmicro-footprints:0402-res, F.Cu at (53.6, 198.4)
- added R170: R_2k2_0402, antmicro-footprints:0402-res, F.Cu at (127.6, 192.2)
- added R171: R_0R_0402, antmicro-footprints:0402-res, F.Cu at (132.1, 192.7)
- added R172: R_2k2_0402, antmicro-footprints:0402-res, F.Cu at (126.6, 192.2)
- added R173: R_2k2_0402, antmicro-footprints:0402-res, F.Cu at (125.6, 192.2)
- added R174: R_0R_0402, antmicro-footprints:0402-res, F.Cu at (122.1, 191.7)
- added R175: R_4k7_0402, antmicro-footprints:0402-res, F.Cu at (93.3, 195.4)
- added R176: R_4k7_0402, antmicro-footprints:0402-res, F.Cu at (99.4, 195.4)
- added R177: R_2k2_0402, antmicro-footprints:0402-res, F.Cu at (124.6, 192.2)
- added R178: R_2k2_0402, antmicro-footprints:0402-res, F.Cu at (123.6, 192.2)
- added R179: R_0R_0402, antmicro-footprints:0402-res, F.Cu at (122.1, 192.7)
- added R18: R_0R_0402, antmicro-footprints:0402-res, F.Cu at (56.2, 202.8)
- added R180: R_100k_0402, antmicro-footprints:0402-res, F.Cu at (83.6, 194.0)
- added R183: R_10k_0402, antmicro-footprints:0402-res, F.Cu at (82.8, 198.9)
- added R184: R_10k_0402, antmicro-footprints:0402-res, F.Cu at (88.8, 199.0)
- added R185: R_4k7_0402, antmicro-footprints:0402-res, F.Cu at (81.0, 195.3)
- added R186: R_4k7_0402, antmicro-footprints:0402-res, F.Cu at (87.0, 195.4)
- added R211: R_0R_0402, antmicro-footprints:0402-res, B.Cu at (116.4, 142.8)
- added R212: R_0R_0402, antmicro-footprints:0402-res, B.Cu at (115.2, 142.8)
- added R213: R_0R_0402, antmicro-footprints:0402-res, B.Cu at (110.4, 142.8)
- added R214: R_0R_0402, antmicro-footprints:0402-res, B.Cu at (109.4, 142.8)
- added R215: R_0R_0402, antmicro-footprints:0402-res, F.Cu at (150.1, 169.7)
- added R216: R_0R_0402, antmicro-footprints:0402-res, F.Cu at (151.7, 171.2)
- added R217: R_0R_0402, antmicro-footprints:0402-res, F.Cu at (145.5, 171.2)
- added R218: R_0R_0402, antmicro-footprints:0402-res, F.Cu at (147.1, 169.7)
- added R219: R_10k2_0402, antmicro-footprints:0402-res, F.Cu at (151.7, 172.2)
- added R220: R_10k_0402, antmicro-footprints:0402-res, F.Cu at (152.2, 193.7)
- added R222: R_100k_0402, antmicro-footprints:0402-res, F.Cu at (134.2, 212.5)
- added R223: R_200R_0402, antmicro-footprints:0402-res, F.Cu at (138.4, 210.3)
- added R224: R_0R_0402, antmicro-footprints:0402-res, F.Cu at (145.5, 172.2)
- added R225: R_0R_0402, antmicro-footprints:0402-res, F.Cu at (145.5, 173.2)
- added R226: R_0R_0402, antmicro-footprints:0402-res, F.Cu at (145.5, 174.2)
- added R227: R_0R_0402, antmicro-footprints:0402-res, F.Cu at (147.1, 175.8)
- added R228: R_0R_0402, antmicro-footprints:0402-res, F.Cu at (149.1, 175.8)
- added R229: R_0R_0402, antmicro-footprints:0402-res, F.Cu at (150.1, 175.8)
- added R230: R_100k_0402, antmicro-footprints:0402-res, F.Cu at (142.2, 212.5)
- added R231: R_200R_0402, antmicro-footprints:0402-res, F.Cu at (146.4, 210.3)
- added R233: R_0R_0603, antmicro-footprints:0603-res, F.Cu at (148.7, 108.7)
- added R234: R_0R_0603, antmicro-footprints:0603-res, F.Cu at (148.7, 111.1)
- added R235: R_0R_0603, antmicro-footprints:0603-res, F.Cu at (148.7, 113.5)
- added R236: R_0R_0402, antmicro-footprints:0402-res, F.Cu at (150.8, 87.9)
- added R237: R_0R_0402, antmicro-footprints:0402-res, F.Cu at (150.8, 88.9)
- added R238: R_0R_0402, antmicro-footprints:0402-res, F.Cu at (150.8, 90.1)
- added R239: R_0R_0402, antmicro-footprints:0402-res, F.Cu at (150.8, 91.1)
- added R240: R_0R_0402, antmicro-footprints:0402-res, F.Cu at (150.8, 83.1)
- added R241: R_0R_0402, antmicro-footprints:0402-res, F.Cu at (150.8, 84.1)
- added R243: R_0R_0402, antmicro-footprints:0402-res, F.Cu at (159.2, 83.7)
- added R244: R_0R_0402, antmicro-footprints:0402-res, F.Cu at (159.2, 84.7)
- added R245: R_0R_0402, antmicro-footprints:0402-res, F.Cu at (159.2, 88.5)
- added R246: R_0R_0402, antmicro-footprints:0402-res, F.Cu at (159.2, 89.5)
- added R247: R_0R_0603, antmicro-footprints:0603-res, F.Cu at (160.6, 111.1)
- added R248: R_0R_0603, antmicro-footprints:0603-res, F.Cu at (160.6, 113.5)
- added R249: R_100k_0402, antmicro-footprints:0402-res, F.Cu at (109.2, 169.3)
- added R250: R_10k_0402, antmicro-footprints:0402-res, F.Cu at (78.6, 178.1)
- added R251: R_10k_0402, antmicro-footprints:0402-res, F.Cu at (78.6, 171.1)
- added R252: R_0R_1206, antmicro-footprints:1206-res, F.Cu at (35.8, 138.6)
- added R253: R_0R_1206, antmicro-footprints:1206-res, F.Cu at (35.8, 141.1)
- added R254: R_10k_0402, antmicro-footprints:0402-res, F.Cu at (80.1, 174.2)
- added R255: R_10k_0402, antmicro-footprints:0402-res, F.Cu at (80.0, 167.2)
- added R256: R_1k_0402, antmicro-footprints:0402-res, F.Cu at (113.5, 174.1)
- added R257: R_200k_0402, antmicro-footprints:0402-res, F.Cu at (112.2, 172.8)
- added R258: R_200k_0402, antmicro-footprints:0402-res, F.Cu at (113.7, 169.3)
- added R259: R_10k_0402, antmicro-footprints:0402-res, F.Cu at (120.8, 174.7)
- added R260: R_0R_0402, antmicro-footprints:0402-res, F.Cu at (120.8, 169.9)
- added R261: R_200k_0402, antmicro-footprints:0402-res, F.Cu at (127.7, 170.7)
- added R262: R_100k_0402, antmicro-footprints:0402-res, F.Cu at (43.1, 163.0)
- added R265: R_5R6_0402, antmicro-footprints:0402-res, F.Cu at (46.3, 163.0)
- added R268: R_0R_0402, antmicro-footprints:0402-res, F.Cu at (83.0, 161.7)
- added R273: R_0R_0603, antmicro-footprints:0603-res, F.Cu at (32.2, 157.6)
- added R276: R_0R_0603, antmicro-footprints:0603-res, F.Cu at (79.0, 157.5)
- added R294: R_2k2_0402, antmicro-footprints:0402-res, B.Cu at (60.8, 62.9)
- added R37: R_47k_0402, antmicro-footprints:0402-res, F.Cu at (51.0, 201.0)
- added R38: R_47k_0402, antmicro-footprints:0402-res, F.Cu at (56.6, 206.0)
- added R40: R_0R_0402, antmicro-footprints:0402-res, F.Cu at (37.3, 190.7)
- added R47: R_10k_0402, antmicro-footprints:0402-res, F.Cu at (37.3, 188.8)
- added R49: R_10k_0402, antmicro-footprints:0402-res, F.Cu at (41.3, 190.3)
- added R60: R_0R_0402, antmicro-footprints:0402-res, F.Cu at (33.2, 174.1)
- added R61: R_0R_0402, antmicro-footprints:0402-res, F.Cu at (33.2, 175.1)
- added R74: R_10k_0402, antmicro-footprints:0402-res, F.Cu at (107.9, 199.1)
- added R76: R_0R_0402, antmicro-footprints:0402-res, F.Cu at (108.1, 195.4)
- added R77: R_10k_0402, antmicro-footprints:0402-res, F.Cu at (108.1, 194.4)
- added R78: R_2k2_0402, antmicro-footprints:0402-res, F.Cu at (106.1, 195.4)
- added S4: B3U-3000PM, antmicro-footprints:B3U-3000P, F.Cu at (114.8, 177.9)
- added S5: B3U-3000PM, antmicro-footprints:B3U-3000P, F.Cu at (123.3, 177.9)
- added TP1: TP_SMD_0_75MM, antmicro-footprints:Testpoint_smd_0_75mm, F.Cu at (-343.2, 36.7)
- added TP10: TP_SMD_0_75MM, antmicro-footprints:Testpoint_smd_0_75mm, F.Cu at (-343.2, 137.6)
- added TP11: TP_SMD_0_75MM, antmicro-footprints:Testpoint_smd_0_75mm, F.Cu at (-343.2, 144.3)
- added TP12: TP_SMD_0_75MM, antmicro-footprints:Testpoint_smd_0_75mm, F.Cu at (-343.2, 153.2)
- added TP13: TP_SMD_0_75MM, antmicro-footprints:Testpoint_smd_0_75mm, F.Cu at (-343.2, 95.0)
- added TP14: TP_SMD_0_75MM, antmicro-footprints:Testpoint_smd_0_75mm, F.Cu at (-343.2, 101.7)
- added TP15: TP_SMD_0_75MM, antmicro-footprints:Testpoint_smd_0_75mm, F.Cu at (-343.2, 146.5)
- added TP16: TP_SMD_0_75MM, antmicro-footprints:Testpoint_smd_0_75mm, F.Cu at (-343.2, 92.7)
- added TP17: TP_SMD_0_75MM, antmicro-footprints:Testpoint_smd_0_75mm, F.Cu at (-343.2, 106.2)
- added TP18: TP_SMD_0_75MM, antmicro-footprints:Testpoint_smd_0_75mm, F.Cu at (-343.2, 90.5)
- added TP19: TP_SMD_0_75MM, antmicro-footprints:Testpoint_smd_0_75mm, F.Cu at (-343.2, 139.8)
- added TP2: TP_SMD_0_75MM, antmicro-footprints:Testpoint_smd_0_75mm, F.Cu at (-343.2, 47.9)
- added TP20: TP_SMD_0_75MM, antmicro-footprints:Testpoint_smd_0_75mm, F.Cu at (-343.2, 119.6)
- added TP21: TP_SMD_0_75MM, antmicro-footprints:Testpoint_smd_0_75mm, F.Cu at (-343.2, 103.9)
- added TP22: TP_SMD_0_75MM, antmicro-footprints:Testpoint_smd_0_75mm, F.Cu at (-343.2, 112.9)
- added TP23: TP_SMD_0_75MM, antmicro-footprints:Testpoint_smd_0_75mm, F.Cu at (-343.2, 110.7)
- added TP24: TP_SMD_0_75MM, antmicro-footprints:Testpoint_smd_0_75mm, F.Cu at (-343.2, 108.4)
- added TP25: TP_SMD_0_75MM, antmicro-footprints:Testpoint_smd_0_75mm, F.Cu at (-343.2, 142.0)
- added TP26: TP_SMD_0_75MM, antmicro-footprints:Testpoint_smd_0_75mm, F.Cu at (-343.2, 99.5)
- added TP27: TP_SMD_0_75MM, antmicro-footprints:Testpoint_smd_0_75mm, F.Cu at (-343.2, 151.0)
- added TP29: TP_SMD_0_75MM, antmicro-footprints:Testpoint_smd_0_75mm, F.Cu at (-343.2, 157.7)
- added TP3: TP_SMD_0_75MM, antmicro-footprints:Testpoint_smd_0_75mm, F.Cu at (-343.2, 45.7)
- added TP30: TP_SMD_0_75MM, antmicro-footprints:Testpoint_smd_0_75mm, F.Cu at (-343.2, 77.1)
- added TP31: TP_SMD_0_75MM, antmicro-footprints:Testpoint_smd_0_75mm, F.Cu at (-343.2, 79.3)
- added TP32: TP_SMD_0_75MM, antmicro-footprints:Testpoint_smd_0_75mm, F.Cu at (-343.2, 83.8)
- added TP33: TP_SMD_0_75MM, antmicro-footprints:Testpoint_smd_0_75mm, F.Cu at (-343.2, 81.5)
- added TP34: TP_SMD_0_75MM, antmicro-footprints:Testpoint_smd_0_75mm, F.Cu at (-343.2, 65.9)
- added TP35: TP_SMD_0_75MM, antmicro-footprints:Testpoint_smd_0_75mm, F.Cu at (-343.2, 74.8)
- added TP36: TP_SMD_0_75MM, antmicro-footprints:Testpoint_smd_0_75mm, F.Cu at (-343.2, 68.1)
- added TP37: TP_SMD_0_75MM, antmicro-footprints:Testpoint_smd_0_75mm, F.Cu at (-343.2, 54.6)
- added TP38: TP_SMD_0_75MM, antmicro-footprints:Testpoint_smd_0_75mm, F.Cu at (-343.2, 61.4)
- added TP39: TP_SMD_0_75MM, antmicro-footprints:Testpoint_smd_0_75mm, F.Cu at (-343.2, 56.9)
- added TP4: TP_SMD_0_75MM, antmicro-footprints:Testpoint_smd_0_75mm, F.Cu at (-343.2, 43.4)
- added TP40: TP_SMD_0_75MM, antmicro-footprints:Testpoint_smd_0_75mm, F.Cu at (-343.2, 63.6)
- added TP41: TP_SMD_0_75MM, antmicro-footprints:Testpoint_smd_0_75mm, F.Cu at (-343.2, 52.4)
- added TP42: TP_SMD_0_75MM, antmicro-footprints:Testpoint_smd_0_75mm, F.Cu at (-343.2, 70.3)
- added TP43: TP_SMD_0_75MM, antmicro-footprints:Testpoint_smd_0_75mm, F.Cu at (-343.2, 72.6)
- added TP44: TP_SMD_0_75MM, antmicro-footprints:Testpoint_smd_0_75mm, F.Cu at (-343.2, 59.1)
- added TP45: TP_SMD_0_75MM, antmicro-footprints:Testpoint_smd_0_75mm, F.Cu at (-343.2, 50.2)
- added TP46: TP_SMD_0_75MM, antmicro-footprints:Testpoint_smd_0_75mm, F.Cu at (-343.2, 86.0)
- added TP47: TP_SMD_0_75MM, antmicro-footprints:Testpoint_smd_0_75mm, F.Cu at (-343.2, 88.3)
- added TP48: TP_SMD_0_75MM, antmicro-footprints:Testpoint_smd_0_75mm, F.Cu at (-343.2, 128.6)
- added TP49: TP_SMD_0_75MM, antmicro-footprints:Testpoint_smd_0_75mm, F.Cu at (-343.2, 97.2)
- added TP5: TP_SMD_0_75MM, antmicro-footprints:Testpoint_smd_0_75mm, F.Cu at (-343.2, 41.2)
- added TP50: TP_SMD_0_75MM, antmicro-footprints:Testpoint_smd_0_75mm, F.Cu at (-343.2, 133.1)
- added TP51: TP_SMD_0_75MM, antmicro-footprints:Testpoint_smd_0_75mm, F.Cu at (-343.2, 117.4)
- added TP52: TP_SMD_0_75MM, antmicro-footprints:Testpoint_smd_0_75mm, F.Cu at (-343.2, 155.5)
- added TP53: TP_SMD_0_75MM, antmicro-footprints:Testpoint_smd_0_75mm, F.Cu at (-343.2, 135.3)
- added TP54: TP_SMD_0_75MM, antmicro-footprints:Testpoint_smd_0_75mm, F.Cu at (-343.2, 148.8)
- added TP55: TP_SMD_0_75MM, antmicro-footprints:Testpoint_smd_0_75mm, F.Cu at (-343.2, 124.1)
- added TP56: TP_SMD_0_75MM, antmicro-footprints:Testpoint_smd_0_75mm, F.Cu at (-343.2, 34.5)
- added TP57: TP_SMD_0_75MM, antmicro-footprints:Testpoint_smd_0_75mm, F.Cu at (-343.2, 39.0)
- added TP6: TP_SMD_0_75MM, antmicro-footprints:Testpoint_smd_0_75mm, F.Cu at (-343.2, 126.4)
- added TP7: TP_SMD_0_75MM, antmicro-footprints:Testpoint_smd_0_75mm, F.Cu at (-343.2, 115.2)
- added TP8: TP_SMD_0_75MM, antmicro-footprints:Testpoint_smd_0_75mm, F.Cu at (-343.2, 130.8)
- added TP9: TP_SMD_0_75MM, antmicro-footprints:Testpoint_smd_0_75mm, F.Cu at (-343.2, 121.9)
- added U2: 74LVC2G07GV, antmicro-footprints:SC-74, F.Cu at (53.6, 205.0)
- added U24: AP22615, antmicro-footprints:TSOT23-6, F.Cu at (92.5, 197.9)
- added U25: AP22615, antmicro-footprints:TSOT23-6, F.Cu at (98.5, 197.9)
- added U26: PCA9547BS, antmicro-footprints:VQFN-24, F.Cu at (128.9, 197.5)
- added U29: AP22615, antmicro-footprints:TSOT23-6, F.Cu at (80.5, 197.9)
- added U3: 74LVC2G07GV, antmicro-footprints:SC-74, F.Cu at (53.6, 201.0)
- added U30: AP22615, antmicro-footprints:TSOT23-6, F.Cu at (86.5, 197.9)
- added U31: NTS0102GT, antmicro-footprints:PSON50P100X195X50-8N, F.Cu at (115.8, 142.8)
- added U32: NTS0102GT, antmicro-footprints:PSON50P100X195X50-8N, F.Cu at (109.8, 142.8)
- added U34: PCAL6408ABSHP, antmicro-footprints:VQFN-16-1EP_3x3mm, F.Cu at (148.6, 172.8)
- added U37: 74LVC2G14GV, antmicro-footprints:SOT23-6L, F.Cu at (114.8, 171.7)
- added U38: 74LVC1G175GV, antmicro-footprints:SOT-23-6, F.Cu at (122.0, 172.3)
- added U41: TPS7B8133DRVR, antmicro-footprints:WSON6_TI_2x2mm, F.Cu at (30.2, 159.6)
- added U42: TPS7A0518PDBVT, antmicro-footprints:SOT-23-5, F.Cu at (80.6, 160.5)
- added U8: TPS7B8133DRVR, antmicro-footprints:WSON6_TI_2x2mm, F.Cu at (56.3, 147.1)
- added U9: AP22615, antmicro-footprints:TSOT23-6, F.Cu at (105.6, 198.0)
- added kibuzzard-633EE390: G***, kibuzzard-633EE390, F.Cu at (31.3, 64.3)
- C102, C103, C145, C146, C147, C148, C149, C150, C151, C152, C153, C154, C155, C156, C157, C158, C159, C160, C161, C162, C26, C28, C30, C33, C35, C53, C58, C59, C92, C93, D1, D16, D17, D19, D21, D22, D23, D35, D4, D5, J9, Q5, Q6, Q7, Q8, R181, R182, R187, R188, R189, R190, R191, R192, R193, R195, R196, R198, R203, R204, R221, R277, R278, R39, R41, R42, R43, R44, R45, R48, R50, R51, R52, R53, R54, R55, R62, R63, R64, R65, R66, R67, R68, R69, R70, R71, SW1, U27, U28, U33, U6, U7: moved to F.Cu
- J7, S1, S2, S3: moved to B.Cu
- moved R14 293.1 mm to (-145.3, -13.0), turned to 0 degrees
- moved R28 292.3 mm to (-145.3, -12.0), turned to 0 degrees
- moved C10 291.0 mm to (-145.4, -10.0), turned to 0 degrees
- moved C9 290.3 mm to (-145.4, -9.00), turned to 0 degrees
- moved R26 283.9 mm to (-145.7, 1.90), turned to -90 degrees
- moved R25 281.9 mm to (-144.7, 1.90), turned to -90 degrees
- moved J1 275.7 mm to (-137.7, -8.45), turned to 90 degrees
- moved C12 274.3 mm to (-133.1, -17.2), turned to 0 degrees
- moved R31 272.3 mm to (-133.2, -14.7), turned to 0 degrees
- moved R30 271.4 mm to (-133.2, -13.7), turned to 0 degrees
- moved R27 269.8 mm to (-133.1, -11.9), turned to 180 degrees
- moved R35 266.9 mm to (-133.3, -7.80), turned to 0 degrees
- moved R36 266.2 mm to (-133.3, -6.80), turned to 0 degrees
- moved R33 265.4 mm to (-133.3, -5.80), turned to 0 degrees
- moved R34 264.7 mm to (-133.3, -4.80), turned to 0 degrees
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