File: jetson-orin-baseboard.kicad_pcb (KiCad board)
At the start: 8 copper layers, 110 x 55 mm, 656 parts, among them IC1 ACPL-217-500E, J1 2199230-6, J10 533980471, J11 LSHM-140-01-L-DH-A-S-TR, J12 Molex_Nano-Fit-105430_xx02-ho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, J13 46756-1001, J2 1-2199230-6, J3 USB4105-GF-A, J4 WE_632723300011_alt_symbol, J5 WE_632723300011_alt_symbol, J6 5-2337992-8, J7 WE_68715014522, J8 WE_68715014522, J9 TC2050-IDC-NL, M1 jetson-orin-nx/nano-module, M2 M2_4222, M3 M2_2280, Q1 NX138BKMYL, Q10 NX138BKMYL, Q11 NX138BKMYL, Q12 NX138BKMYL, Q13 BCM857BS-7-F, Q14 BCM857BS-7-F, Q15 SSM3J332R, Q16 SSM3J332R, Q17 NX138BKMYL, Q18 SSM3J332R, Q19 NX138BKMYL, Q2 NX138BKMYL, Q20 NX138BKMYL, Q21 NX138BKMYL, Q22 NX138BKMYL, Q3 NX138BKMYL, Q4 NX138BKMYL, Q5 NX138BKMYL, Q6 NX138BKMYL, Q7 NX138BKMYL, Q8 NX138BKMYL, Q9 NX138BKMYL, SW1 PCM12SMTR, U1 74LVC1T45GM, U10 TUSB1046-DCI, U11 TPD4E05U06QDQARQ1, U12 AP22615, U13 TPD4E05U06QDQARQ1, U14 TPD4E05U06QDQARQ1, U15 TPD4E05U06QDQARQ1, U16 TPD4E05U06QDQARQ1, U17 HD3SS3220, U18 AP22615, U19 TPD4E05U06QDQARQ1, U2 74LVC2G07GV, U20 TPD4E05U06QDQARQ1, U21 TPD4E05U06QDQARQ1, U22 TPS2372-3RGWR, U23 ULS-12/5-D48N-C, U24 AP22653FDZ-7, U25 AP22653FDZ-7, U26 PCA9547BS, U27 AP22653FDZ-7, U28 AP22653FDZ-7, U29 TPD4E05U06QDQARQ1, U3 74LVC2G07GV, U31 NTS0102GT, U32 NTS0102GT, U33 NTS0102GT, U34 PCAL6408ABSHP, U37 74LVC2G14GV, U38 74LVC1G175GV, U39 MP2386GG-P, U4 NTS0102GT, U40 MP2386GG-P, U41 TPS7B8133DRVR, U42 TPS7A0518PDBVT, U43 NTS0102GT, U44 TPD4E02B04DQA, U45 TPD4E02B04DQA, U46 TPD4E02B04DQA, U5 FT230XQ-R, U6 TPS65988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

Commit message: Rearanged PCB to move M.2 connector and changed exp conn resistors to res arrays
Parts:
- removed C131: C_2u2_0402, antmicro-footprints:0402-cap
- removed C165, C166: C_4u7_0402, antmicro-footprints:0402-cap
- removed C86: C_100n_0402_16V, antmicro-footprints:0402-cap
- removed D16, D17, D19, D21, D22, D23: LTST-C190GKT, antmicro-footprints:LED_0603
- removed the J13 at (94.2, 125.5)
- removed the J4 at (75.0, 125.8)
- removed the J4 at (113.7, 125.8)
- removed Q5, Q6, Q7, Q8: NX138BKMYL, antmicro-footprints:DFN1006-3
- removed R191, R193, R195, R198, R203, R204: R_200R_0402, antmicro-footprints:0402-res
- removed R192, R196: R_100k_0402, antmicro-footprints:0402-res
- removed R224, R225, R226, R227, R236, R237, R238, R239, R240, R241, R243, R244, R245, R246: R_0R_0402, antmicro-footprints:0402-res
- removed R302, R303, R304, R305, R306, R307, R308, R309, R310, R311, R312, R313, R314, R315, R316, R317, R318, R319, R320, R321, R322, R323, R324, R325, R326, R327, R328, R329, R330, R331, R332, R333, R334: R_470R_0603, antmicro-footprints:0603-res
- added C51: C_10u_0603, antmicro-footprints:0603-cap, F.Cu at (101.8, 170.8)
- added C52: C_100n_0402_50V, antmicro-footprints:0402-cap, F.Cu at (109.2, 175.7)
- added C83: C_22u_0402, antmicro-footprints:0402-cap, F.Cu at (109.2, 170.5)
- added R100: 4x330R_0402_array, antmicro-footprints:R_Array_4x0402, B.Cu at (87.8, 96.3)
- added R101: 4x330R_0402_array, antmicro-footprints:R_Array_4x0402, B.Cu at (90.5, 93.7)
- added R102: 4x330R_0402_array, antmicro-footprints:R_Array_4x0402, B.Cu at (93.2, 93.7)
- added R120: R_0R_0402, antmicro-footprints:0402-res, B.Cu at (87.8, 104.0)
- added R121: R_0R_0402, antmicro-footprints:0402-res, B.Cu at (87.8, 103.0)
- added R53: 4x330R_0402_array, antmicro-footprints:R_Array_4x0402, B.Cu at (99.0, 93.8)
- added R54: 4x330R_0402_array, antmicro-footprints:R_Array_4x0402, B.Cu at (101.8, 93.8)
- added R55: R_0R_0402, antmicro-footprints:0402-res, B.Cu at (106.2, 93.9)
- added R62: R_0R_0402, antmicro-footprints:0402-res, B.Cu at (107.2, 93.9)
- added R63: 4x330R_0402_array, antmicro-footprints:R_Array_4x0402, B.Cu at (104.5, 93.8)
- added R64: 4x330R_0402_array, antmicro-footprints:R_Array_4x0402, B.Cu at (87.8, 99.0)
- added TP35: TP_SMD_0_75MM, antmicro-footprints:Testpoint_smd_0_75mm, F.Cu at (100.8, 176.1)
- added U30: TPD4E05U06QDQARQ1, antmicro-footprints:USON-10_2.5x1.0mm_P0.5mm, B.Cu at (170.3, 124.8)
- C44, C48, D39, D40, D41, D42, D43, D44, D45, D46, D47, D48, D49, D50, R39, U29: moved to B.Cu
- D1: value KP-1608CGCK -> LTST-C190GKT; moved to B.Cu
- D15: value KP-1608CGCK -> LTST-C190GKT
- R140, R197, R206: value R_470R_0603 -> R_470R_0402; footprint antmicro-footprints:0603-res -> antmicro-footprints:0402-res
- R25: value R_0R_0402 -> 4x0R_0201_array; footprint antmicro-footprints:0402-res -> antmicro-footprints:EXB18V
- R26: value R_0R_0402 -> 4x330R_0402_array; footprint antmicro-footprints:0402-res -> antmicro-footprints:R_Array_4x0402; moved to B.Cu
- R335, R336: value R_470R_0603 -> R_470R_0402; footprint antmicro-footprints:0603-res -> antmicro-footprints:0402-res; moved to B.Cu
- moved R39 314.9 mm to (112.7, 95.0), turned to 180 degrees
- moved D1 314.5 mm to (112.5, 96.6), turned to 0 degrees
- moved C44 221.3 mm to (163.0, 104.5), turned to 90 degrees
- moved D45 217.7 mm to (162.7, 110.5), turned to 90 degrees
- moved D40 216.3 mm to (160.1, 110.5), turned to 90 degrees
- moved D47 216.3 mm to (166.4, 104.1), turned to 90 degrees
- moved D39 215.8 mm to (162.0, 107.0), turned to 90 degrees
- moved D50 214.7 mm to (156.1, 110.5), turned to 90 degrees
- moved D41 213.9 mm to (164.5, 99.8), turned to 90 degrees
- moved D46 213.5 mm to (166.8, 97.0), turned to 90 degrees
- moved D44 212.7 mm to (164.9, 96.3), turned to 90 degrees
- moved D49 211.8 mm to (159.4, 99.8), turned to 90 degrees
- moved D48 210.8 mm to (159.7, 96.3), turned to 90 degrees
- moved D43 210.4 mm to (157.9, 96.3), turned to 90 degrees
- moved C48 210.4 mm to (155.0, 100.2), turned to 90 degrees
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Connections:
- net /USB Debug, DP/USBC0_CONN_RX1_N renamed /USB Debug, DP/USBC0_RX1_N
- net /USB Debug, DP/USBC0_CONN_RX1_P renamed /USB Debug, DP/USBC0_RX1_P
- net /USB Debug, DP/USBC0_CONN_RX2_N renamed /USB Debug, DP/USBC0_RX2_N
- net /USB Debug, DP/USBC0_CONN_RX2_P renamed /USB Debug, DP/USBC0_RX2_P
- A1 pad 94: HDMI_CEC -> Net-(A1-Pad94)
- D4 pad 2: unconnected-(D4-Pad2) -> GND
- D5 pad 2: unconnected-(D5-Pad2) -> GND
- J1 pad 3: /M.2/M2_E_USB_D_P -> USB2_D_P
- J1 pad 5: /M.2/M2_E_USB_D_N -> USB2_D_N
- J11 pad 15: /Peripherals/PCIE2_CLK_CONN_N -> PCIE2_CLK_N
- J11 pad 17: /Peripherals/PCIE2_CLK_CONN_P -> PCIE2_CLK_P
- J11 pad 18: /Peripherals/PCIE3_CLK_CONN_N -> PCIE3_CLK_N
- J11 pad 20: /Peripherals/PCIE3_CLK_CONN_P -> PCIE3_CLK_P
- J11 pad 21: /Peripherals/USBSS2_RX_CONN_N -> USBSS2_RX_N
- J11 pad 23: /Peripherals/USBSS2_RX_CONN_P -> USBSS2_RX_P
- J11 pad 27: Net-(J11-Pad27) -> /Peripherals/PCIE2_RST_CONN*
- J11 pad 29: Net-(J11-Pad29) -> /Peripherals/PCIE2_CLKREQ_CONN*
- J11 pad 3: /Peripherals/PCIE2_RX0_CONN_N -> PCIE2_RX0_N
- J11 pad 30: Net-(J11-Pad30) -> PCIE3_RST_CONN*
- J11 pad 31: Net-(J11-Pad31) -> /Peripherals/GPIO01_CONN
- J11 pad 32: Net-(J11-Pad32) -> /Peripherals/PCIE3_CLKREQ_CONN*
- J11 pad 33: Net-(J11-Pad33) -> /Peripherals/GPIO07_CONN
- J11 pad 34: Net-(J11-Pad34) -> /Peripherals/PCIE_WAKE_SEL_EXT_CONN
- J11 pad 35: Net-(J11-Pad35) -> /Peripherals/GPIO09_CONN
- J11 pad 36: Net-(J11-Pad36) -> /Peripherals/GPIO13_CONN
- J11 pad 39: Net-(J11-Pad39) -> /Peripherals/GPIO10_CONN
- J11 pad 40: Net-(J11-Pad40) -> /Peripherals/GPIO12_CONN
- J11 pad 41: Net-(J11-Pad41) -> /Peripherals/UART1_TXD_CONN
- J11 pad 42: Net-(J11-Pad42) -> /Peripherals/GPIO11_CONN
- J11 pad 43: Net-(J11-Pad43) -> /Peripherals/UART1_RXD_CONN
- J11 pad 44: Net-(J11-Pad44) -> /Peripherals/GPIO00_CONN
- J11 pad 45: Net-(J11-Pad45) -> /Peripherals/I2S0_SDIN_CONN
- J11 pad 46: Net-(J11-Pad46) -> /Peripherals/I2S0_SCLK_CONN
- J11 pad 47: Net-(J11-Pad47) -> /Peripherals/I2S0_LRCK_CONN
- J11 pad 48: Net-(J11-Pad48) -> /Peripherals/I2S0_SDOUT_CONN
- J11 pad 5: /Peripherals/PCIE2_RX0_CONN_P -> PCIE2_RX0_P
- J11 pad 51: Net-(J11-Pad51) -> /Peripherals/SPIO_SCK_CONN
- J11 pad 52: Net-(J11-Pad52) -> /Peripherals/SPI1_SCK_CONN
- J11 pad 53: Net-(J11-Pad53) -> /Peripherals/SPIO_MOSI_CONN
- J11 pad 54: Net-(J11-Pad54) -> /Peripherals/SPI1_MOSI_CONN
- J11 pad 55: Net-(J11-Pad55) -> /Peripherals/SPIO_MISO_CONN
- J11 pad 56: Net-(J11-Pad56) -> /Peripherals/SPI1_MISO_CONN
- J11 pad 57: Net-(J11-Pad57) -> /Peripherals/~{SPI0_CS0_CONN}
- J11 pad 58: Net-(J11-Pad58) -> /Peripherals/~{SPI1_CS0_CONN}
- J11 pad 59: Net-(J11-Pad59) -> /Peripherals/~{SPI0_CS1_CONN}
- J11 pad 6: /Peripherals/PCIE2_RX1_CONN_N -> PCIE2_RX1_N
- J11 pad 60: Net-(J11-Pad60) -> /Peripherals/~{SPI1_CS1_CONN}
- J11 pad 8: /Peripherals/PCIE2_RX1_CONN_P -> PCIE2_RX1_P
- J11 pad S1: unconnected-(J11-PadS1) -> GND
- J11 pad S2: unconnected-(J11-PadS2) -> GND
- R25 pad 1: /M.2/M2_E_USB_D_P -> CSIA_PEN
- R25 pad 2: USB2_D_P -> CSIB_PEN
- R26 pad 1: /M.2/M2_E_USB_D_N -> /Peripherals/GPIO07_CONN
- R26 pad 2: USB2_D_N -> /Peripherals/GPIO01_CONN
- U29 pad 1: /Peripherals/USBSS2_RX_CONN_N -> USBSS2_RX_N
- U29 pad 10: /Peripherals/USBSS2_RX_CONN_N -> USBSS2_RX_N
- U29 pad 2: /Peripherals/USBSS2_RX_CONN_P -> USBSS2_RX_P
- U29 pad 9: /Peripherals/USBSS2_RX_CONN_P -> USBSS2_RX_P
