File: ethernet.kicad_sch (KiCad schematic)
At the start: 37 parts, among them IC1 ACPL-217-500E, J6 5-2337992-8, U22 TPS2372-3RGWR, U23 ULS-12{slash}5-D48N-C

Commit message: Loclib
Parts:
- C52: footprint antmicro-footprints:0402-cap -> jetson-orin-baseboard-footprints:0402-cap; symbol antmicroCapacitorsmisc:C_100n_0402_50V -> jetson-orin-baseboard:C_100n_0402_50V
- C76: footprint antmicro-footprints:0805-cap -> jetson-orin-baseboard-footprints:0805-cap; symbol antmicroCapacitorsmisc:C_100n_0805_100V -> jetson-orin-baseboard:C_100n_0805_100V
- C77: footprint antmicro-footprints:0402-cap -> jetson-orin-baseboard-footprints:0402-cap; symbol antmicroCapacitors0402:C_10n_0402 -> jetson-orin-baseboard:C_10n_0402
- C78: footprint antmicro-footprints:0402-cap -> jetson-orin-baseboard-footprints:0402-cap; symbol antmicroCapacitors0402:C_100n_0402 -> jetson-orin-baseboard:C_100n_0402
- C79, C80, C81, C82: footprint antmicro-footprints:2220-cap -> jetson-orin-baseboard-footprints:2220-cap; symbol antmicroCapacitorsmisc:C_22u_2220_100V -> jetson-orin-baseboard:C_22u_2220_100V
- C84, C85: footprint antmicro-footprints:1206-cap -> jetson-orin-baseboard-footprints:1206-cap; symbol antmicroCapacitorsmisc:C_47u_16V_1206 -> jetson-orin-baseboard:C_47u_16V_1206
- D12, D13: footprint antmicro-footprints:DFN3538 -> jetson-orin-baseboard-footprints:DFN3538; symbol antmicroTVSDiodes:CD-MMBL110S -> jetson-orin-baseboard:CD-MMBL110S
- D14: footprint antmicro-footprints:SOD-123F -> jetson-orin-baseboard-footprints:SOD-123F; symbol antmicroDiodesRectifiersSingle:PTVS58VS1UR,115 -> jetson-orin-baseboard:PTVS58VS1UR,115
- D15: footprint antmicro-footprints:LED_0603 -> jetson-orin-baseboard-footprints:LED_0603; symbol antmicroLEDIndicationDiscrete:LTST-C190GKT -> jetson-orin-baseboard:LTST-C190GKT
- FB2, FB3: footprint antmicro-footprints:0805-res -> jetson-orin-baseboard-footprints:0805-res; symbol antmicroFerriteBeadsandChips:BLM21PG221SN1D -> jetson-orin-baseboard:BLM21PG221SN1D
- IC1: footprint antmicro-footprints:SOIC127P700X242-4N -> jetson-orin-baseboard-footprints:SOIC127P700X242-4N; symbol antmicroOptoisolatorsLogicOutput:ACPL-217-500E -> jetson-orin-baseboard:ACPL-217-500E
- J6: footprint antmicro-footprints:5-2337992-8 -> jetson-orin-baseboard-footprints:5-2337992-8; symbol antmicroModularConnectorsJacksWithMagnetics:5-2337992-8 -> jetson-orin-baseboard:5-2337992-8
- R123: footprint antmicro-footprints:0402-res -> jetson-orin-baseboard-footprints:0402-res; symbol antmicroResistors0402:R_1k3_0402 -> jetson-orin-baseboard:R_1k3_0402
- R129, R148: footprint antmicro-footprints:0402-res -> jetson-orin-baseboard-footprints:0402-res; symbol antmicroResistors0402:R_0R_0402 -> jetson-orin-baseboard:R_0R_0402
- R130: footprint antmicro-footprints:0402-res -> jetson-orin-baseboard-footprints:0402-res; symbol antmicroResistors0402:R_63R4_0402 -> jetson-orin-baseboard:R_63R4_0402
- R142: footprint antmicro-footprints:0402-res -> jetson-orin-baseboard-footprints:0402-res; symbol antmicroResistors0402:R_49k9_0402 -> jetson-orin-baseboard:R_49k9_0402
- R145: footprint antmicro-footprints:0402-res -> jetson-orin-baseboard-footprints:0402-res; symbol antmicroResistors0402:R_1k2_0402 -> jetson-orin-baseboard:R_1k2_0402
- R146: footprint antmicro-footprints:0402-res -> jetson-orin-baseboard-footprints:0402-res; symbol antmicroResistors0402:R_24k9_0402 -> jetson-orin-baseboard:R_24k9_0402
- R147: footprint antmicro-footprints:0402-res -> jetson-orin-baseboard-footprints:0402-res; symbol antmicroResistors0402:R_200R_0402 -> jetson-orin-baseboard:R_200R_0402
- R149, R150, R153: footprint antmicro-footprints:0402-res -> jetson-orin-baseboard-footprints:0402-res; symbol antmicroResistors0402:R_10k_0402 -> jetson-orin-baseboard:R_10k_0402
- R151, R152: footprint antmicro-footprints:0402-res -> jetson-orin-baseboard-footprints:0402-res; symbol antmicroResistors0402:R_220R_0402 -> jetson-orin-baseboard:R_220R_0402
- R154: footprint antmicro-footprints:0402-res -> jetson-orin-baseboard-footprints:0402-res; symbol antmicroResistors0402:R_32k4_0402 -> jetson-orin-baseboard:R_32k4_0402
- R155, R156: footprint antmicro-footprints:0603-res -> jetson-orin-baseboard-footprints:0603-res; symbol antmicroResistors0603:R_1k_0603 -> jetson-orin-baseboard:R_1k_0603
- R157: footprint antmicro-footprints:0603-res -> jetson-orin-baseboard-footprints:0603-res; symbol antmicroResistors0603:R_0R_0603 -> jetson-orin-baseboard:R_0R_0603
- U22: footprint antmicro-footprints:Texas_RGW0020B -> jetson-orin-baseboard-footprints:Texas_RGW0020B; symbol antmicroPMICPowerDistributionSwitchesLoadDrivers:TPS2372-3RGWR -> jetson-orin-baseboard:TPS2372-3RGWR
- U23: footprint antmicro-footprints:ULS-12_5-D48N-C -> jetson-orin-baseboard-footprints:ULS-12_5-D48N-C; symbol antmicroDCDCConverters:ULS-12{brace}slash}5-D48N-C -> jetson-orin-baseboard:ULS-12{brace}slash}5-D48N-C
Connections:
- net VSS: no longer FB3.2
- net at D12.1, D13.1: no longer FB3.1
