File: jetson-orin-baseboard.kicad_sch (KiCad schematic)
At the start: 4 parts

Commit message: Loclib
Parts:
- SP1, SP2, SP3, SP4: footprint antmicro-footprints:9774060151 -> jetson-orin-baseboard-footprints:9774060151; symbol antmicroMechanicalParts:9774060151 -> jetson-orin-baseboard:9774060151
