File: usb.kicad_sch (KiCad schematic)
At the start: 123 parts, among them J3 USB4105-GF-A, J4 WE_632723300011_alt_symbol, U10 TUSB1046-DCI, U11 TPD4E05U06QDQARQ1, U12 AP22615, U13 TPD4E05U06QDQARQ1, U14 TPD4E05U06QDQARQ1, U15 TPD4E05U06QDQARQ1, U16 TPD4E05U06QDQARQ1, U5 FT230XQ-R, U6 TPS65988, U7 W25Q80DVUXIE_TR, U8 NCP730BMT330TBG, U9 AP22615

Commit message: Add capacitors to USB SS. Add VBUS, _HV 1u/4u7 caps. Improve readability
Parts:
- removed R195, R196, R198, R199, R80, R81: R_0R_0402, jetson-orin-baseboard-footprints:0402-res, symbol jetson-orin-baseboard:R_0R_0402
- added C? (x2): C_4u7_0402_25V, antmicro-footprints:0402-cap, symbol antmicroCapacitors0402:C_4u7_0402_25V
- added C? (x4): C_100n_0402, jetson-orin-baseboard-footprints:0402-cap, symbol jetson-orin-baseboard:C_100n_0402
- added C? (x2): C_1u_0402_16V, antmicro-footprints:0402-cap, symbol antmicroCapacitors0402:C_1u_0402_16V
- added C? (x2): C_47p_0402, antmicro-footprints:0402-cap, symbol antmicroCapacitors0402:C_47p_0402
- added C?: C_10u_0402, jetson-orin-baseboard-footprints:0402-cap, symbol jetson-orin-baseboard:C_10u_0402
- added R? (x2): R_27R_0402, antmicro-footprints:0402-res, symbol antmicroResistors0402:R_27R_0402
- R59: DNP (none) -> DNP
Connections:
- net +3V3: now also C?.1
- net FTDI_3V3: now also R46.1; no longer R46.2
- net GND: now also C?.2, C?.2, C?.2, C?.2, C?.2, C?.2, C?.2
- net PDC_I2C3_SCL: now also R66.2, U6.21 (I2C3_SCL/GPIO5)
- net USBC0_VBUS: now also C?.1
- net USBC3_D_N: now also C?.1, R?.2
- net USBC3_D_P: now also C?.1, R?.2
- net USBC3_VBUS: now also C?.1
- net USBPD1_HV: now also C?.1
- net USBPD2_HV: now also C?.1
- net USBSS0_RX_C_N: now also C?.2
- net USBSS0_RX_C_P: now also C?.2
- net USBSS0_RX_N: now also C?.1
- net USBSS0_RX_P: now also C?.1
- net USBSS0_TX_C_N: now also C?.2
- net USBSS0_TX_C_P: now also C?.2
- net USBSS0_TX_N: now also C?.1
- net USBSS0_TX_P: now also C?.1
- net USB_FTDI_N: now also R?.1
- net USB_FTDI_P: now also R?.1
- net at C31.1, U5.9 (~{RESET}): now also R46.2; no longer R46.1
Other:
- moved on the sheet: C26, C27, C28, C29, C30, C31, C32, C34, C35, C36, C37, C45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
