File: som.kicad_sch (KiCad schematic)
At the start: 34 parts, among them M1 jetson-orin-nx/nano-module, U4 NTS0102GT

Commit message: Loclib
Parts:
- C1, C2, C3, C38, C39, C4, C46: footprint antmicro-footprints:0603-cap -> jetson-orin-baseboard-footprints:0603-cap; symbol antmicroCapacitors0603:C_22u_0603_16V -> jetson-orin-baseboard:C_22u_0603_16V
- S1: footprint antmicro-footprints:SW_SPST_4.2x2.8 -> jetson-orin-baseboard-footprints:SW_SPST_4.2x2.8; symbol antmicroPushbuttonSwitches:KMR2 -> jetson-orin-baseboard:KMR2
Changed lines of the file:
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@@
     (pin "1")
   )
-  (symbol (lib_id "antmicroPushbuttonSwitches:KMR2") (at 129.54 126.365 270) (unit 1)
+  (symbol (lib_id "jetson-orin-baseboard:KMR2") (at 129.54 126.365 270) (unit 1)
     (in_bom yes) (on_board yes) (fields_autoplaced)
     (property "Reference" "S1" (id 0) (at 132.969 125.5303 90)
@@
       (effects (font (size 1.27 1.27)) (justify left))
     )
-    (property "Footprint" "antmicro-footprints:SW_SPST_4.2x2.8" (id 2) (at 134.62 131.445 0)
+    (property "Footprint" "jetson-orin-baseboard-footprints:SW_SPST_4.2x2.8" (id 2) (at 134.62 131.445 0)
       (effects (font (size 1.27 1.27)) (justify left) hide)
     )
@@
     (pin "2")
   )
-  (symbol (lib_id "antmicroCapacitors0603:C_22u_0603_16V") (at 38.735 97.79 0) (unit 1)
+  (symbol (lib_id "jetson-orin-baseboard:C_22u_0603_16V") (at 38.735 97.79 0) (unit 1)
     (in_bom yes) (on_board yes)
     (property "Reference" "C38" (id 0) (at 39.37 95.25 0)
@@
       (effects (font (size 1.27 1.27)) hide)
     )
-    (property "Footprint" "antmicro-footprints:0603-cap" (id 2) (at 43.815 92.71 0)
+    (property "Footprint" "jetson-orin-baseboard-footprints:0603-cap" (id 2) (at 43.815 92.71 0)
       (effects (font (size 1.524 1.524)) (justify left) hide)
     )
@@
     (pin "1")
   )
-  (symbol (lib_id "antmicroCapacitors0603:C_22u_0603_16V") (at 27.94 97.79 0) (unit 1)
+  (symbol (lib_id "jetson-orin-baseboard:C_22u_0603_16V") (at 27.94 97.79 0) (unit 1)
     (in_bom yes) (on_board yes)
     (property "Reference" "C3" (id 0) (at 28.575 95.25 0)
@@
       (effects (font (size 1.27 1.27)) hide)
     )
-    (property "Footprint" "antmicro-footprints:0603-cap" (id 2) (at 33.02 92.71 0)
+    (property "Footprint" "jetson-orin-baseboard-footprints:0603-cap" (id 2) (at 33.02 92.71 0)
       (effects (font (size 1.524 1.524)) (justify left) hide)
     )
@@
     (pin "1")
   )
-  (symbol (lib_id "antmicroCapacitors0603:C_22u_0603_16V") (at 17.145 97.79 0) (mirror y) (unit 1)
+  (symbol (lib_id "jetson-orin-baseboard:C_22u_0603_16V") (at 17.145 97.79 0) (mirror y) (unit 1)
     (in_bom yes) (on_board yes)
     (property "Reference" "C1" (id 0) (at 17.78 95.25 0)
@@
       (effects (font (size 1.27 1.27)) hide)
     )
-    (property "Footprint" "antmicro-footprints:0603-cap" (id 2) (at 12.065 92.71 0)
+    (property "Footprint" "jetson-orin-baseboard-footprints:0603-cap" (id 2) (at 12.065 92.71 0)
       (effects (font (size 1.524 1.524)) (justify left) hide)
     )
@@
     (pin "1")
   )
-  (symbol (lib_id "antmicroCapacitors0603:C_22u_0603_16V") (at 27.94 113.03 0) (unit 1)
+  (symbol (lib_id "jetson-orin-baseboard:C_22u_0603_16V") (at 27.94 113.03 0) (unit 1)
     (in_bom yes) (on_board yes)
     (property "Reference" "C4" (id 0) (at 28.575 110.49 0)
@@
       (effects (font (size 1.27 1.27)) hide)
     )
-    (property "Footprint" "antmicro-footprints:0603-cap" (id 2) (at 33.02 107.95 0)
+    (property "Footprint" "jetson-orin-baseboard-footprints:0603-cap" (id 2) (at 33.02 107.95 0)
       (effects (font (size 1.524 1.524)) (justify left) hide)
     )
@@
     (pin "2")
   )
-  (symbol (lib_id "antmicroCapacitors0603:C_22u_0603_16V") (at 38.735 113.03 0) (unit 1)
+  (symbol (lib_id "jetson-orin-baseboard:C_22u_0603_16V") (at 38.735 113.03 0) (unit 1)
     (in_bom yes) (on_board yes)
     (property "Reference" "C39" (id 0) (at 39.37 110.49 0)
@@
       (effects (font (size 1.27 1.27)) hide)
     )
-    (property "Footprint" "antmicro-footprints:0603-cap" (id 2) (at 43.815 107.95 0)
+    (property "Footprint" "jetson-orin-baseboard-footprints:0603-cap" (id 2) (at 43.815 107.95 0)
       (effects (font (size 1.524 1.524)) (justify left) hide)
     )
@@
     (pin "1")
   )
-  (symbol (lib_id "antmicroCapacitors0603:C_22u_0603_16V") (at 17.145 113.03 0) (mirror y) (unit 1)
+  (symbol (lib_id "jetson-orin-baseboard:C_22u_0603_16V") (at 17.145 113.03 0) (mirror y) (unit 1)
     (in_bom yes) (on_board yes)
     (property "Reference" "C2" (id 0) (at 17.78 110.49 0)
@@
       (effects (font (size 1.27 1.27)) hide)
     )
-    (property "Footprint" "antmicro-footprints:0603-cap" (id 2) (at 12.065 107.95 0)
+    (property "Footprint" "jetson-orin-baseboard-footprints:0603-cap" (id 2) (at 12.065 107.95 0)
       (effects (font (size 1.524 1.524)) (justify left) hide)
     )
@@
     (pin "2")
   )
-  (symbol (lib_id "antmicroCapacitors0603:C_22u_0603_16V") (at 49.53 113.03 0) (unit 1)
+  (symbol (lib_id "jetson-orin-baseboard:C_22u_0603_16V") (at 49.53 113.03 0) (unit 1)
     (in_bom yes) (on_board yes)
     (property "Reference" "C46" (id 0) (at 50.165 110.49 0)
@@
       (effects (font (size 1.27 1.27)) hide)
     )
-    (property "Footprint" "antmicro-footprints:0603-cap" (id 2) (at 54.61 107.95 0)
-      (effects (font (size 1.524 1.524)) (justify left) hide)
-    )
+    (property "Footprint" "jetson-orin-baseboard-footprints:0603-cap" (id 2) (at 54.61 107.95 0)
+      (effects (font (size 1.524 1.524)) (justify left) hide)
+    )
